Commit message: add go straight line planner

File: ros_model/my_model/urdf/my_pi.xacro (robot description, xacro)
@@ -39,6 +39,6 @@
         <gazebo reference="wheel_${number}">
             <material>Gazebo/Gray</material>
-            <mu1>1000</mu1>
-            <mu2>1000</mu2>
+            <mu1>100</mu1>
+            <mu2>100</mu2>
         </gazebo>
         <transmission name="simple_trans_${number}">

File: ros_model/my_model/urdf/my_pi_with_rplidar.xacro (robot description, xacro)
@@ -7,4 +7,11 @@
 	<xacro:property name="rplidar_offset_z" value="0.07" />
 	<my_robot/>
+	<!-- rplidar -->
+	<joint name="rplidar_joint" type="fixed">
+		<origin xyz="${rplidar_offset_x} ${rplidar_offset_y} ${rplidar_offset_z}" rpy="0 0 0" />
+		<parent link="base_link"/>
+		<child link="laser_link"/>
+	</joint>
+	<rplidar/>
     <gazebo>
     <plugin name="differential_drive_controller" filename="libgazebo_ros_diff_drive.so">
@@ -15,5 +22,5 @@
         <wheelSeparation>0.34</wheelSeparation>
         <wheelDiameter>0.08</wheelDiameter>
-        <torque>50</torque>
+        <torque>100</torque>
         <commandTopic>cmd_vel</commandTopic>
         <odometryTopic>odom</odometryTopic>

File: ros_model/my_model/urdf/rplidar.xacro (robot description, xacro)
@@ -27,4 +27,35 @@
 			<material>Gazebo/Black</material>
 		</gazebo>
+		<gazebo reference="laser_link">
+			<sensor type="ray" name="rplidar">
+				<pose>0 0 0 0 0 0</pose>
+				<visualize>false</visualize>
+				<update_rate>5.5</update_rate>
+				<ray>
+					<scan>
+						<horizontal>
+							<samples>360</samples>
+							<resolution>1</resolution>
+							<min_angle>-3</min_angle>
+							<max_angle>3</max_angle>
+						</horizontal>
+					</scan>
+					<range>
+						<min>0.15</min>
+						<max>6.0</max>
+						<resolution>0.01</resolution>
+					</range>
+					<noise>
+						<type>gaussian</type>
+						<mean>0.0</mean>
+						<stddev>0.01</stddev>
+					</noise>
+				</ray>
+				<plugin name="gazebo_rplidar" filename="libgazebo_ros_laser.so">
+					<topicName>/scan</topicName>
+					<frameName>laser_link</frameName>
+				</plugin>
+			</sensor>
+		</gazebo>
 	</xacro:macro>
 </robot>
